Commit message: Made the simulation start at unstable position

File: urdf/inverted_pendulum.urdf (robot description, URDF)
Before this commit: robot inverted_pendulum, 5 links, 4 joints
Joints:
- joint pendulum_gantry: origin xyz=0.036 0.0 0.062 rpy=0.0 0.0 0.0 -> xyz=0.036 0.0 0.058 rpy=0.3 0.0 0.0

Commit message: Adjusted some values Added robot_state and joint_state publishers to check the integrity of the model in rviz

File: urdf/inverted_pendulum.urdf (robot description, URDF)
Before this commit: robot inverted_pendulum, 5 links, 4 joints
Joints:
- joint pendulum_gantry: origin xyz=0.036 0.0 0.058 rpy=0.3 0.0 0.0 -> xyz=0.036 0.0 0.063 rpy=0.3 0.0 0.0

Commit message: Adjusted the joint positions of the pendulum

File: urdf/inverted_pendulum.urdf (robot description, URDF)
Before this commit: robot inverted_pendulum, 5 links, 4 joints
Links:
- link gantry_assembly: geometry collision mesh filename=package://inverted_pendulum_description/meshes/Gantry_Pendu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; visual mesh filename=package://inverted_pendulum_description/meshes/Gantry_Pendu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
Joints:
- joint base_link_joint: origin xyz=0 0 0 rpy=0 0 0 -> xyz=0 0 1.0 rpy=0 0 0
- joint moving_gantry: origin xyz=0.0 0.0 1.023 -> xyz=0.0 0.0 0.05
- joint pendulum_gantry: origin xyz=0.036 0.0 0.063 rpy=0.3 0.0 0.0 -> xyz=0.03118 0.0 0.0175 rpy=0.3 0.0 0.0
